Commit message: added docs

File: src/unitree_go2_description/xacro/constants.xacro (robot description, xacro)
@@ -26,5 +26,4 @@
     <xacro:property name="leg_offset_x" value="0.1934"/>
     <xacro:property name="leg_offset_y" value="0.0465"/>
-    <!-- <xacro:property name="trunk_offset_z" value="0.01675"/> -->
     <xacro:property name="hip_offset" value="0.0955"/>
     <!-- offset of link locations (left front) -->

File: src/unitree_go2_description/xacro/unitree_go2.xacro (robot description, xacro)
@@ -1,4 +1,5 @@
 <?xml version="1.0"?>
 <robot name="go2" xmlns:xacro="http://www.ros.org/wiki/xacro">
+    <!-- DEBUG mode: Set to 'true' to fix robot to world frame for testing kinematics without physics simulation -->
     <xacro:arg name="DEBUG" default="false"/>
     <xacro:include filename="$(find unitree_go2_description)/xacro/constants.xacro"/>
@@ -7,5 +8,5 @@
     <xacro:include filename="$(find unitree_go2_description)/xacro/gazebo.xacro"/>
     <xacro:include filename="$(find unitree_go2_description)/xacro/lidar.xacro"/>
-    <!-- Debug mode will fix the robot to the world -->
+    <!-- When DEBUG is true, fix the robot to world frame for kinematic testing -->
     <xacro:if value="$(arg DEBUG)">
         <link name="world"/>
